File: Hardware/kicad-project/connectors.kicad_sch (KiCad schematic)
At the start: 24 parts, among them CN10 Conn_02x17_Odd_Even, CN7 Conn_02x10_Odd_Even, CN8 Conn_02x08_Odd_Even, CN9 Conn_02x15_Odd_Even, J1 Brake connector, J2 Conn_01x08, J5 UART Connector, J6 Stepper supply, Q1 Q_NMOS_DGS, Q2 Q_NMOS_DGS

Commit message: hw: update schematic (printable version)
Parts:
- removed CN10: Conn_02x17_Odd_Even, Connector_PinHeader_2.54mm:PinHeader_2x17_P2.54mm_Vertical, symbol Connector_Generic:Conn_02x17_Odd_Even
- removed CN7: Conn_02x10_Odd_Even, Connector_PinHeader_2.54mm:PinHeader_2x10_P2.54mm_Vertical, symbol Connector_Generic:Conn_02x10_Odd_Even
- removed CN8: Conn_02x08_Odd_Even, Connector_PinHeader_2.54mm:PinHeader_2x08_P2.54mm_Vertical, symbol Connector_Generic:Conn_02x08_Odd_Even
- removed CN9: Conn_02x15_Odd_Even, Connector_PinHeader_2.54mm:PinHeader_2x15_P2.54mm_Vertical, symbol Connector_Generic:Conn_02x15_Odd_Even
- removed D1, D5: DIODE, Diode_SMD:D_SOD-323, symbol Simulation_SPICE:DIODE
- removed D7, D8: LED, LED_SMD:LED_0603_1608Metric, symbol Device:LED
- removed J1: Brake connector, Connector_PinHeader_2.54mm:PinHeader_1x02_P2.54mm_Vertical, symbol Connector_Generic:Conn_01x02
- removed J2: Conn_01x08, Connector_PinHeader_2.54mm:PinHeader_1x08_P2.54mm_Vertical, symbol Connector_Generic:Conn_01x08
- removed J5: UART Connector, Connector_PinHeader_2.54mm:PinHeader_1x02_P2.54mm_Vertical, symbol Connector_Generic:Conn_01x02
- removed J6: Stepper supply, Connector_PinHeader_2.54mm:PinHeader_1x02_P2.54mm_Vertical, symbol Connector_Generic:Conn_01x02
- removed Q1, Q2: Q_NMOS_DGS, Package_TO_SOT_SMD:TO-252-2, symbol Device:Q_NMOS_GDS
- removed R1, R28: 10k, Resistor_SMD:R_0603_1608Metric, symbol Device:R
- removed R18: 510, Resistor_SMD:R_0603_1608Metric, symbol Device:R
- removed R19: 330, Resistor_SMD:R_0603_1608Metric, symbol Device:R
- removed R3, R5: 47, Resistor_SMD:R_0603_1608Metric, symbol Device:R
- removed R4: 0, Resistor_SMD:R_0603_1608Metric, symbol Device:R
- removed TP2: TORQUE, TestPoint:TestPoint_Pad_D2.0mm, symbol Connector:TestPoint
- removed TP3: 12V, TestPoint:TestPoint_Pad_D2.0mm, symbol Connector:TestPoint
- removed TP5: BRAKE, TestPoint:TestPoint_Pad_D2.0mm, symbol Connector:TestPoint
Connections:
- no-connect marks 94 -> 0
Other:
- note removed: "BLACK"
- note removed: "BROWN"
- note removed: "GREY"
- note removed: "LED"
- note removed: "PWM BRAKE CONTROLLER"
- note removed: "TESTPOINTS"
- note removed: "TORQUE SENSOR CONNECTOR"
- note removed: "The output Vref is a constant 2.5V output and represents the virtual zero point for direct +/- torque measurement."
- note removed: "UART & STEPPER CONNECTORS"
- note removed: "WHITE"
- note removed: "ZIO CONNECTORS"
