File: Hardware/kicad-project/stepper_testbench.kicad_pcb (KiCad board)
At the start: 2 copper layers, 67.7 x 78.4 mm, 76 parts, among them CN10 Conn_02x17_Odd_Even, CN7 Conn_02x10_Odd_Even, CN8 Conn_02x08_Odd_Even, CN9 Conn_02x15_Odd_Even, J1 Brake connector, J2 Conn_01x08, J4 Conn_01x02, J5 UART Connector, J6 Stepper supply, Q1 Q_NMOS_DGS, Q2 Q_NMOS_DGS, U1 LM358P, U2 LEM-CAS-6NP, U3 LM358P, U4 LM358P, U5 LM7812_TO220, U6 L7805

Commit message: hw: update schematic (printable version)
Parts:
- removed CN10: Conn_02x17_Odd_Even, Connector_PinHeader_2.54mm:PinHeader_2x17_P2.54mm_Vertical
- removed CN7: Conn_02x10_Odd_Even, Connector_PinHeader_2.54mm:PinHeader_2x10_P2.54mm_Vertical
- removed CN8: Conn_02x08_Odd_Even, Connector_PinHeader_2.54mm:PinHeader_2x08_P2.54mm_Vertical
- removed CN9: Conn_02x15_Odd_Even, Connector_PinHeader_2.54mm:PinHeader_2x15_P2.54mm_Vertical
- removed J6: Stepper supply, Connector_PinHeader_2.54mm:PinHeader_1x02_P2.54mm_Vertical
- removed TP5: BRAKE, TestPoint:TestPoint_Pad_D2.0mm
- added CN1: Conn_02x08_Odd_Even, Connector_PinHeader_2.54mm:PinHeader_2x08_P2.54mm_Vertical, F.Cu at (130.2, 105.7)
- added CN2: Conn_02x15_Odd_Even, Connector_PinHeader_2.54mm:PinHeader_2x15_P2.54mm_Vertical, F.Cu at (115.8, 105.7)
- added CN3: Conn_02x17_Odd_Even, Connector_PinHeader_2.54mm:PinHeader_2x17_P2.54mm_Vertical, F.Cu at (108.6, 105.7)
- added CN4: Conn_02x10_Odd_Even, Connector_PinHeader_2.54mm:PinHeader_2x10_P2.54mm_Vertical, F.Cu at (123.0, 105.7)
- added J3: Torque, Connector_PinHeader_2.54mm:PinHeader_1x08_P2.54mm_Vertical, F.Cu at (137.4, 105.7)
- added TP1: 12V, TestPoint:TestPoint_Pad_D2.0mm, F.Cu at (108.3, 150.7)
- C1: value 100n -> 0.33u_DNP; footprint Capacitor_SMD:C_0603_1608Metric -> Capacitor_THT:CP_Radial_D5.0mm_P2.50mm
- C10: value 0.33u -> DNP; footprint Capacitor_SMD:C_0603_1608Metric -> Capacitor_SMD:C_0805_2012Metric
- C11, C12: value 0.1u -> 100n
- C13: value 0.33u_DNP -> C_DNP; footprint Capacitor_THT:CP_Radial_D5.0mm_P2.50mm -> Capacitor_SMD:C_0805_2012Metric
- C14, C16: value 0.1u_DNP -> C_DNP; footprint Capacitor_THT:CP_Radial_D5.0mm_P2.50mm -> Capacitor_SMD:C_0805_2012Metric
- C15: value 0.33u_DNP -> 100n; footprint Capacitor_THT:CP_Radial_D5.0mm_P2.50mm -> Capacitor_SMD:C_0603_1608Metric
- C17, C18, C19: value C -> 0.1u; footprint Capacitor_SMD:C_0805_2012Metric -> Capacitor_SMD:C_0603_1608Metric
- C2: value 0.1u -> 0.33u
- C4: value 100n -> 0.1u_DNP; footprint Capacitor_SMD:C_0603_1608Metric -> Capacitor_THT:CP_Radial_D5.0mm_P2.50mm
- C5: value 0.1u -> 0.33u_DNP; footprint Capacitor_SMD:C_0603_1608Metric -> Capacitor_THT:CP_Radial_D5.0mm_P2.50mm
- C6: value 100n -> 0.33u
- C8: value 0.33u -> 0.1u_DNP; footprint Capacitor_SMD:C_0603_1608Metric -> Capacitor_THT:CP_Radial_D5.0mm_P2.50mm
- C9: value DNP -> 0.1u; footprint Capacitor_SMD:C_0805_2012Metric -> Capacitor_SMD:C_0603_1608Metric
- D1: value DIODE -> LED_GN; footprint Diode_SMD:D_SOD-323 -> LED_SMD:LED_0603_1608Metric
- D2: value DIODE -> LED_RD; footprint Diode_SMD:D_SOD-323 -> LED_SMD:LED_0603_1608Metric
- D3: value D_Zener -> DIODE; footprint Diode_SMD:D_SMA -> Diode_SMD:D_SOD-323
- D4: value LED_RED -> D_Zener; footprint LED_SMD:LED_0603_1608Metric -> Diode_SMD:D_SMA
- D5: value DIODE -> LED_RED; footprint Diode_SMD:D_SOD-323 -> LED_SMD:LED_0603_1608Metric
- D7, D8: value LED -> DIODE; footprint LED_SMD:LED_0603_1608Metric -> Diode_SMD:D_SOD-323
- J1: value Brake connector -> Conn_01x02
- J2: value Conn_01x08 -> UART; footprint Connector_PinHeader_2.54mm:PinHeader_1x08_P2.54mm_Vertical -> Connector_PinHeader_2.54mm:PinHeader_1x02_P2.54mm_Vertical
- J4: value Conn_01x02 -> Stepper supply
- J5: value UART Connector -> Brake
- R1: value 10k -> 330
- R10: value 330k -> 0_DNP
- R11: value 620k -> 0_DNP
- R12, R28, R9: value 10k -> 0
- R13, R8: value 620k -> 10k
- R14: value 100k -> 10k
- R15: value 0 -> 620k
- R16: value R -> 100k
- R17: value R -> 330k
- R18: value 510 -> 620k
- R19: value 330 -> R_DNP
- R2: value 0 -> 510
- R20: value 5k1 -> 0_DNP
- R21: value 1k -> R_DNP
- R23: value R -> 0
- R24: value R -> 10k
- R25: value 0 -> 330k
- R26: value R -> 620k
- R27: value R -> R_DNP
- R3: value 47 -> 5k1
- R4: value 0 -> 47
- R5: value 47 -> 10k
- R6: value 10k -> 1k
- R7: value 330k -> 47
- TP3: value 12V -> BRAKE
- U1: value LM358P -> LM7812_TO220; footprint Package_DIP:DIP-8_W7.62mm -> Package_TO_SOT_THT:TO-220-3_Vertical
- U2: value LEM-CAS-6NP -> L7805; footprint Sensing lib:LEM-CAS-6-NP -> Package_TO_SOT_THT:TO-220-3_Vertical
- U4: value LM358P -> LM35P
- U5: value LM7812_TO220 -> LM35P; footprint Package_TO_SOT_THT:TO-220-3_Vertical -> Package_DIP:DIP-8_W7.62mm
- U6: value L7805 -> LM35P; footprint Package_TO_SOT_THT:TO-220-3_Vertical -> Package_DIP:DIP-8_W7.62mm
Connections:
- C1 pad 1: Net-(C1-Pad1) -> +24V
- C10 pad 1: +12V -> /Sensing/CURRENT_SENSOR_OUTPUT
- C11 pad 1: +5V -> Net-(C11-Pad1)
- C12 pad 1: +12V -> Net-(C12-Pad1)
- C13 pad 1: +24V -> / Power management and peripherals/VOLTAGE_STEPPER_ADC
- C13 pad 2: GND -> Net-(C13-Pad2)
- C14 pad 1: +12V -> / Power management and peripherals/TORQUE_ADC
- C14 pad 2: GND -> Net-(C14-Pad2)
- C15 pad 1: +12V -> Net-(C15-Pad1)
- C16 pad 1: +5V -> / Power management and peripherals/CURRENT_ADC
- C16 pad 2: GND -> Net-(C16-Pad2)
- C17 pad 1: /Sensing/CURRENT_BUFF_ADC -> +5V
- C17 pad 2: /Sensing/CURRENT_BUFF_IN2- -> GND
- C18 pad 1: /Sensing/TORQUE_BUFF_ADC -> +5V
- C18 pad 2: /Sensing/TORQUE_BUFF_IN2- -> GND
- C19 pad 1: /Sensing/VOLTAGE_STEPPER_BUFF_ADC -> +24V
- C19 pad 2: /Sensing/VOLTAGE_STEPPER_BUFF_IN2- -> GND
- C2 pad 1: +5V -> +24V
- C3 pad 1: +5V -> +12V
- C4 pad 1: Net-(C4-Pad1) -> +12V
- C5 pad 1: +5V -> +12V
- C6 pad 1: Net-(C6-Pad1) -> +12V
- C7 pad 1: +24V -> +5V
- C8 pad 1: +24V -> +5V
- C9 pad 1: /Sensing/CURRENT_SENSOR_OUTPUT -> +5V
- D1 pad 2: /Connectors/24V_BRAKE -> / Power management and peripherals/LED2
- D2 pad 2: +24V -> / Power management and peripherals/LED1
- D3 pad 1: +24V -> Net-(D3-Pad1)
- D3 pad 2: GND -> +24V
- D4 pad 1: Net-(D4-Pad1) -> +24V
- D4 pad 2: +24V -> GND
- D5 pad 1: +24V -> Net-(D5-Pad1)
- D5 pad 2: /Connectors/24V_BRAKE -> +24V
- D7 pad 2: /Connectors/LED1 -> / Power management and peripherals/24V_BRAKE
- D8 pad 1: Net-(D8-Pad1) -> +24V
- D8 pad 2: /Connectors/LED2 -> / Power management and peripherals/24V_BRAKE
- FB1 pad 1: /Power/VIN -> / Power management and peripherals/VIN
- FB1 pad 2: Net-(D2-Pad1) -> Net-(D3-Pad1)
- J1 pad 1: /Connectors/24V_BRAKE -> GND
- J1 pad 2: Net-(D1-Pad1) -> / Power management and peripherals/VIN
- J2 pad 1: +12V -> / Power management and peripherals/UART1_TX
- J2 pad 2: +12V -> / Power management and peripherals/UART1_RX
- J4 pad 1: GND -> / Power management and peripherals/STEPPER+
- J4 pad 2: /Power/VIN -> / Power management and peripherals/STEPPER-
- J5 pad 1: /Connectors/UART1_TX -> / Power management and peripherals/24V_BRAKE
- J5 pad 2: /Connectors/UART1_RX -> Net-(D7-Pad1)
- Q1 pad 2: Net-(Q1-Pad2) -> / Power management and peripherals/STEPPER-
- R1 pad 1: GND -> Net-(D1-Pad1)
- R1 pad 2: Net-(Q1-Pad1) -> GND
- R10 pad 1: Net-(C4-Pad1) -> +24V
- R10 pad 2: /Sensing/ADC_TORQUE -> /Sensing/V_SUPPLY_BUFF
- R11 pad 1: /Sensing/ADC_TORQUE -> / Power management and peripherals/TORQUE
- R11 pad 2: GND -> /Sensing/TORQUE_BUFF
- R12 pad 1: Net-(C6-Pad1) -> Net-(R12-Pad1)
- R12 pad 2: /Sensing/V_SUPPLY_BUFF -> /Sensing/CURRENT_SENSOR_OUTPUT
- R13 pad 1: Net-(C6-Pad1) -> Net-(C11-Pad1)
- R13 pad 2: /Sensing/ADC_V_SUPPLY -> /Sensing/V_SUPPLY_BUFF
- R14 pad 1: /Sensing/ADC_V_SUPPLY -> Net-(C12-Pad1)
- R14 pad 2: GND -> /Sensing/TORQUE_BUFF
- R15 pad 1: /Sensing/CURRENT_SENSOR_OUTPUT -> Net-(C11-Pad1)
- R15 pad 2: /Sensing/CURRENT_BUFF -> /Sensing/ADC_V_SUPPLY
- R16 pad 1: /Sensing/CURRENT_BUFF_IN2- -> /Sensing/ADC_V_SUPPLY
- R17 pad 1: /Sensing/CURRENT_BUFF_IN2- -> Net-(C12-Pad1)
- R17 pad 2: /Sensing/CURRENT_BUFF_ADC -> /Sensing/ADC_TORQUE
- R18 pad 1: Net-(D7-Pad1) -> /Sensing/ADC_TORQUE
- R19 pad 1: Net-(D8-Pad1) -> Net-(C13-Pad2)
- R2 pad 1: Net-(R2-Pad1) -> Net-(D2-Pad1)
- R2 pad 2: /Sensing/CURRENT_SENSOR_OUTPUT -> GND
- R20 pad 1: Net-(D4-Pad1) -> /Sensing/CURRENT_SENSOR_OUTPUT
- R20 pad 2: GND -> /Sensing/CURRENT_BUFF
- R21 pad 1: Net-(D6-Pad1) -> Net-(C14-Pad2)
- R22 pad 1: /Sensing/TORQUE_BUFF -> Net-(C13-Pad2)
- R22 pad 2: /Connectors/TORQUE -> / Power management and peripherals/VOLTAGE_STEPPER_ADC
- R23 pad 1: /Sensing/TORQUE_BUFF_IN2- -> Net-(C14-Pad2)
- R23 pad 2: GND -> / Power management and peripherals/TORQUE_ADC
- R24 pad 1: /Sensing/TORQUE_BUFF_IN2- -> Net-(C15-Pad1)
- R24 pad 2: /Sensing/TORQUE_BUFF_ADC -> /Sensing/CURRENT_BUFF
- R25 pad 1: /Sensing/V_SUPPLY_BUFF -> Net-(C15-Pad1)
- R25 pad 2: +24V -> /Sensing/ADC_CURRENT
- R26 pad 1: /Sensing/VOLTAGE_STEPPER_BUFF_IN2- -> /Sensing/ADC_CURRENT
- R27 pad 1: /Sensing/VOLTAGE_STEPPER_BUFF_IN2- -> Net-(C16-Pad2)
- R27 pad 2: /Sensing/VOLTAGE_STEPPER_BUFF_ADC -> GND
- R28 pad 1: GND -> Net-(C16-Pad2)
- R28 pad 2: Net-(Q2-Pad1) -> / Power management and peripherals/CURRENT_ADC
- R3 pad 1: /Connectors/PWM_BRAKE -> Net-(D5-Pad1)
- R3 pad 2: Net-(Q1-Pad1) -> GND
- R4 pad 1: Net-(Q1-Pad2) -> / Power management and peripherals/EN_STEPPER_SUPPLY
- R4 pad 2: Net-(D1-Pad1) -> Net-(Q1-Pad1)
- R5 pad 1: /Connectors/ENABLE_STEPPER_SUPPLY -> GND
- R5 pad 2: Net-(Q2-Pad1) -> Net-(Q1-Pad1)
- R6 pad 1: Net-(C1-Pad1) -> Net-(D6-Pad1)
- R6 pad 2: /Sensing/CURRENT_BUFF -> GND
- R7 pad 1: Net-(C1-Pad1) -> / Power management and peripherals/PWM_BRAKE
- R7 pad 2: /Sensing/ADC_CURRENT -> Net-(Q2-Pad1)
- R8 pad 1: /Sensing/ADC_CURRENT -> GND
- R8 pad 2: GND -> Net-(Q2-Pad1)
- R9 pad 1: Net-(C4-Pad1) -> Net-(Q2-Pad2)
- R9 pad 2: /Sensing/TORQUE_BUFF -> Net-(D7-Pad1)
- TP2 pad 1: /Connectors/TORQUE -> / Power management and peripherals/TORQUE
- TP3 pad 1: +12V -> / Power management and peripherals/PWM_BRAKE
- U1 pad 1: /Sensing/CURRENT_BUFF -> +24V
- U1 pad 2: /Sensing/CURRENT_BUFF -> GND
- U1 pad 3: /Sensing/CURRENT_SENSOR_OUTPUT -> +12V
- U2 pad 1: +5V -> +12V
- U2 pad 3: Net-(R2-Pad1) -> +5V
- U4 pad 6: /Sensing/VOLTAGE_STEPPER_BUFF_IN2- -> Net-(C13-Pad2)
- U4 pad 7: /Sensing/VOLTAGE_STEPPER_BUFF_ADC -> / Power management and peripherals/VOLTAGE_STEPPER_ADC
- U5 pad 1: +24V -> /Sensing/TORQUE_BUFF
- U5 pad 2: GND -> /Sensing/TORQUE_BUFF
- U5 pad 3: +12V -> / Power management and peripherals/TORQUE
- U6 pad 1: +12V -> /Sensing/CURRENT_BUFF
- U6 pad 2: GND -> /Sensing/CURRENT_BUFF
- U6 pad 3: +5V -> /Sensing/CURRENT_SENSOR_OUTPUT
Routing:
- net / Power management and peripherals/24V_BRAKE: track 0.00 -> 66.7 mm
- net /Sensing/TORQUE_BUFF: track 15.1 -> 81.0 mm, vias 0 -> 1
- net +12V: track 75.3 -> 10.2 mm, vias 2 -> 0
- net /Connectors/UART1_RX: track 54.6 -> 0.00 mm
- net GND: track 1.46 -> 54.0 mm, vias 96 -> 99
- net Net-(D7-Pad1): track 4.45 -> 54.6 mm, vias 1 -> 0
- net /Connectors/UART1_TX: track 49.7 -> 0.00 mm
- net / Power management and peripherals/TORQUE: track 0.00 -> 48.6 mm, vias 0 -> 2
- net /Sensing/CURRENT_BUFF_ADC: track 46.6 -> 0.00 mm, vias 1 -> 0
- net /Sensing/ADC_TORQUE: track 13.4 -> 51.1 mm, vias 0 -> 2
- net /Connectors/TORQUE: track 35.3 -> 0.00 mm, vias 2 -> 0
- net /Sensing/CURRENT_SENSOR_OUTPUT: track 43.2 -> 75.3 mm, vias 3 -> 2
- net /Sensing/VOLTAGE_STEPPER_BUFF_ADC: track 29.1 -> 0.00 mm
- net Net-(D5-Pad1): track 0.00 -> 20.9 mm, vias 0 -> 1
- net /Connectors/PWM_BRAKE: track 20.9 -> 0.00 mm, vias 1 -> 0
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- added copper zone on F.Cu, net / Power management and peripherals/EN_STEPPER_SUPPLY
- removed copper zone on F.Cu, net Net-(Q1-Pad2)

Commit message: hw: add note to layout and add pdf
Parts:
- U3: value LM358P -> LEM-CAS-6NP; footprint Package_DIP:DIP-8_W7.62mm -> Sensing lib:CAS-6-NP
- moved TP1 100.3 mm to (159.5, 64.5)
- moved CN7 83.3 mm to (180.8, 45.7)
- moved CN10 79.3 mm to (180.8, 72.9)
- moved J2 65.4 mm to (177.0, 48.5), turned to 180 degrees
- moved C13 51.2 mm to (213.4, 82.9)
- moved CN8 50.9 mm to (135.1, 55.1)
- moved C15 49.3 mm to (205.3, 101.3)
- moved U5 47.0 mm to (171.7, 105.7), turned to 180 degrees
- moved C14 38.3 mm to (203.4, 84.8)
- moved U6 35.3 mm to (152.2, 104.4), turned to 180 degrees
- moved J3 35.0 mm to (171.4, 113.7), turned to -90 degrees
- moved U3 34.7 mm to (148.6, 79.8), turned to -90 degrees
- moved CN9 33.8 mm to (135.1, 78.0)
- moved U1 32.3 mm to (166.9, 58.9), turned to 0 degrees
- moved J4 32.0 mm to (137.4, 50.0), turned to 180 degrees
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- renumbered CN3 to CN10, CN4 to CN7, CN1 to CN8, CN2 to CN9
Connections:
- U3 pad 1: /Sensing/TORQUE_BUFF -> +5V
- U3 pad 2: /Sensing/TORQUE_BUFF -> GND
- U3 pad 3: /Connectors/TORQUE -> Net-(R12-Pad1)
- U3 pad 4: GND -> +24V
- U3 pad 5: /Sensing/ADC_TORQUE -> +24V
- U3 pad 6: /Sensing/TORQUE_BUFF_IN2- -> +24V
- U3 pad 7: /Sensing/TORQUE_BUFF_ADC -> / Power management and peripherals/STEPPER+
- U3 pad 8: +5V -> / Power management and peripherals/STEPPER+
Routing:
- net +12V: track 10.2 -> 116.8 mm, vias 0 -> 2
- net / Power management and peripherals/CURRENT_ADC: track 5.61 -> 79.9 mm, vias 0 -> 1
- net /Sensing/CURRENT_SENSOR_OUTPUT: track 75.3 -> 4.25 mm, vias 2 -> 1
- net /Sensing/TORQUE_BUFF: track 81.0 -> 15.1 mm, vias 1 -> 0
- net Net-(D7-Pad1): track 54.6 -> 0.00 mm
- net / Power management and peripherals/UART1_RX: track 0.00 -> 54.6 mm
- net / Power management and peripherals/24V_BRAKE: track 66.7 -> 17.0 mm
- net / Power management and peripherals/UART1_TX: track 0.00 -> 49.7 mm
- net /Sensing/TORQUE_BUFF_ADC: track 44.3 -> 0.00 mm
- net / Power management and peripherals/TORQUE_ADC: track 0.00 -> 44.3 mm
- net +5V: track 73.4 -> 112.0 mm, vias 2 -> 5
- net /Connectors/STEPPER+: track 34.3 -> 0.00 mm
- net / Power management and peripherals/STEPPER+: track 0.00 -> 34.3 mm
- net /Sensing/ADC_TORQUE: track 51.1 -> 17.8 mm, vias 2 -> 1
- net GND: track 54.0 -> 29.2 mm, vias 99 -> 96
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Other:
- board text added: "NOTE: usare il layout alla versione 0.1 su git. Qui avendo aggiornato lo schematico è necessario rioridnare condensatori e resistenze. Da sistemare: - label bottom torque connector - FOOTPRINT DIODI - V_supply_Buff track width 1mm - DRILL connettori da allargare"
- board text removed: "Check footprint of zener diode"
