File: Hardware/kicad-project/stepper_testbench.kicad_pcb (KiCad board)
At the start: 2 copper layers, 67.7 x 78.4 mm, 76 parts, among them CN10 Conn_02x17_Odd_Even, CN7 Conn_02x10_Odd_Even, CN8 Conn_02x08_Odd_Even, CN9 Conn_02x15_Odd_Even, J1 Brake connector, J2 Conn_01x08, J4 Conn_01x02, J5 UART Connector, J6 Stepper supply, Q1 Q_NMOS_DGS, Q2 Q_NMOS_DGS, U1 LM358P, U2 LEM-CAS-6NP, U3 LM358P, U4 LM358P, U5 LM7812_TO220, U6 L7805

Commit message: initial commit
Other:
- board text removed: "Check footprint of zener diode"
Changed lines of the file:
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@@
     (effects (font (size 1 1) (thickness 0.15)) (justify mirror))
   )
-  (gr_text "GND\n" (at 166.066 110.773 90) (layer "B.SilkS")
-    (effects (font (size 1 0.8) (thickness 0.15)) (justify mirror))
-  )
-  (gr_text "TRQ\n" (at 158.516 110.773 90) (layer "B.SilkS")
-    (effects (font (size 1 0.8) (thickness 0.15)) (justify mirror))
-  )
-  (gr_text "12V" (at 153.416 110.848 90) (layer "B.SilkS")
+  (gr_text "GND\n" (at 158.514 110.827 90) (layer "B.SilkS")
+    (effects (font (size 1 0.8) (thickness 0.15)) (justify mirror))
+  )
+  (gr_text "TRQ\n" (at 166.064 110.827 90) (layer "B.SilkS")
+    (effects (font (size 1 0.8) (thickness 0.15)) (justify mirror))
+  )
+  (gr_text "12V" (at 171.164 110.752 90) (layer "B.SilkS")
     (effects (font (size 1 0.8) (thickness 0.15)) (justify mirror))
   )
@@
     (effects (font (size 1 1) (thickness 0.15)) (justify mirror))
   )
-  (gr_text "GND\n" (at 163.516 110.773 90) (layer "B.SilkS")
+  (gr_text "GND\n" (at 161.064 110.827 90) (layer "B.SilkS")
     (effects (font (size 1 0.8) (thickness 0.15)) (justify mirror))
   )
@@
     (effects (font (size 1 1) (thickness 0.15)) (justify mirror))
   )
-  (gr_text "TRQ\n" (at 161.066 110.748 90) (layer "B.SilkS")
+  (gr_text "TRQ\n" (at 163.514 110.852 90) (layer "B.SilkS")
     (effects (font (size 1 0.8) (thickness 0.15)) (justify mirror))
   )
@@
     (effects (font (size 0.9 1) (thickness 0.225)) (justify mirror))
   )
-  (gr_text "NC" (at 168.741 111.023 90) (layer "B.SilkS")
-    (effects (font (size 1 1) (thickness 0.15)) (justify mirror))
-  )
-  (gr_text "NC" (at 171.166 110.998 90) (layer "B.SilkS")
+  (gr_text "NC" (at 155.839 110.577 90) (layer "B.SilkS")
+    (effects (font (size 1 1) (thickness 0.15)) (justify mirror))
+  )
+  (gr_text "NC" (at 153.414 110.602 90) (layer "B.SilkS")
     (effects (font (size 1 1) (thickness 0.15)) (justify mirror))
   )
@@
     (effects (font (size 0.9 1) (thickness 0.225)) (justify mirror))
   )
-  (gr_text "12V" (at 155.991 110.823 90) (layer "B.SilkS")
+  (gr_text "12V" (at 168.589 110.777 90) (layer "B.SilkS")
     (effects (font (size 1 0.8) (thickness 0.15)) (justify mirror))
   )
@@
   )
   (gr_text "TORQUE" (at 176.276 116.586) (layer "F.SilkS")
-    (effects (font (size 1 1) (thickness 0.15)))
-  )
-  (gr_text "Check footprint \nof zener diode" (at 159.512 27.432) (layer "User.5")
     (effects (font (size 1 1) (thickness 0.15)))
   )
@@
   (via (at 127.936 102.915) (size 0.55) (drill 0.25) (layers "F.Cu" "B.Cu") (free) (net 5))
   (via (at 166.07 49.81) (size 0.55) (drill 0.25) (layers "F.Cu" "B.Cu") (free) (net 5))
-  (via (at 157.34 111) (size 0.55) (drill 0.25) (layers "F.Cu" "B.Cu") (free) (net 5))
+  (via (at 167.24 110.6) (size 0.55) (drill 0.25) (layers "F.Cu" "B.Cu") (free) (net 5))
   (via (at 154.178 100.838) (size 0.55) (drill 0.25) (layers "F.Cu" "B.Cu") (free) (net 5))
   (via (at 151.8 77.06) (size 0.55) (drill 0.25) (layers "F.Cu" "B.Cu") (free) (net 5))

Commit message: clean repo
Parts:
- D1, D2, D5: footprint Diode_SMD:D_SOD-323 -> Diode_SMD:D_0805_2012Metric
