File: Hardware/kicad-project/stepper_testbench.kicad_sch (KiCad schematic)
At the start: 0 parts

Commit message: hw: update schematic (printable version)
Other:
- sheet Power renamed  Power management and peripherals
- removed sheet Connectors
- sheet  Power management and peripherals: file power.kicad_sch -> power_and_peripherals.kicad_sch
- sheet  Power management and peripherals ports: added CURRENT_ADC, STEPPER+, TORQUE, TORQUE_ADC, VOLTAGE_STEPPER_ADC; removed none
- title: (none) -> STB

Commit message: hw: add heading to the schematic
Other:
- company: (none) -> ProM Facility 
- title: STB -> STB - Expansion Board
Changed lines of the file:
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@@
   (paper "A4")
   (title_block
-    (title "STB")
+    (title "STB - Expansion Board")
     (date "2022-08-09")
     (rev "0.2")
+    (company "ProM Facility ")
   )
   (wire (pts (xy 135.001 87.884) (xy 165.481 87.884))
